File: hardware/prototype/trivial-double/trivial-double.kicad_pcb (KiCad board)
At the start: 2 copper layers, 24.1 x 15.2 mm, 4 parts, among them P1 CONN_02X01, SW1 SWITCH_INV

Commit message: Increased trace and via diameter size
Routing:
- net Net-(P1-Pad2): track 27.6 -> 24.7 mm
- net Net-(P1-Pad1): track 10.3 -> 9.21 mm
Other:
- net class Default: trace_width 0.4 -> 0.5; via_dia 0.6 -> 1.5; via_drill 0.4 -> 1
- rule trace_min: 0.2 -> 0.5
- rule via_min_drill: 0.3 -> 1
- rule via_min_size: 0.4 -> 1.5
Changed lines of the file:
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@@
   (general
     (links 5)
-    (no_connects 0)
+    (no_connects 5)
     (area 114.224999 93.904999 140.56512 110.649)
     (thickness 1.6)
     (drawings 4)
-    (tracks 20)
+    (tracks 15)
     (zones 0)
     (modules 4)
@@
   )
   (setup
-    (last_trace_width 0.4)
+    (last_trace_width 0.5)
     (trace_clearance 0.4)
     (zone_clearance 0.508)
     (zone_45_only no)
-    (trace_min 0.2)
+    (trace_min 0.5)
     (segment_width 0.2)
     (edge_width 0.15)
-    (via_size 0.6)
-    (via_drill 0.4)
-    (via_min_size 0.4)
-    (via_min_drill 0.3)
+    (via_size 1.5)
+    (via_drill 1)
+    (via_min_size 1.5)
+    (via_min_drill 1)
     (uvia_size 0.3)
     (uvia_drill 0.1)
@@
   (net_class Default "This is the default net class."
     (clearance 0.4)
-    (trace_width 0.4)
-    (via_dia 0.6)
-    (via_drill 0.4)
+    (trace_width 0.5)
+    (via_dia 1.5)
+    (via_drill 1)
     (uvia_dia 0.3)
     (uvia_drill 0.1)
@@
   (gr_line (start 138.43 109.22) (end 114.3 109.22) (layer Edge.Cuts) (width 0.15))
   (gr_line (start 138.43 93.98) (end 138.43 109.22) (layer Edge.Cuts) (width 0.15))
-  (segment (start 119.38 101.981) (end 122.809 105.41) (width 0.4) (layer B.Cu) (net 1))
-  (segment (start 122.809 105.41) (end 127 105.41) (width 0.4) (layer B.Cu) (net 1))
-  (segment (start 129.54 105.41) (end 134.62 105.41) (width 0.4) (layer B.Cu) (net 2))
-  (segment (start 134.62 105.41) (end 135.89 106.68) (width 0.4) (layer B.Cu) (net 2))
-  (segment (start 124.46 96.52) (end 120.142 96.52) (width 0.4) (layer B.Cu) (net 3))
-  (segment (start 120.142 96.52) (end 119.38 97.282) (width 0.4) (layer B.Cu) (net 3))
-  (segment (start 128.27 96.52) (end 124.46 96.52) (width 0.4) (layer F.Cu) (net 3))
-  (via (at 124.46 96.52) (size 0.6) (drill 0.4) (layers F.Cu B.Cu) (net 3))
-  (segment (start 120.142 96.52) (end 119.38 97.282) (width 0.4) (layer F.Cu) (net 3))
-  (segment (start 124.46 100.33) (end 124.160001 100.030001) (width 0.4) (layer B.Cu) (net 4))
-  (segment (start 124.160001 100.030001) (end 118.563397 100.030001) (width 0.4) (layer B.Cu) (net 4))
-  (segment (start 117.509999 103.139999) (end 119.38 105.01) (width 0.4) (layer B.Cu) (net 4))
-  (segment (start 118.563397 100.030001) (end 117.509999 101.083399) (width 0.4) (layer B.Cu) (net 4))
-  (segment (start 117.509999 101.083399) (end 117.509999 103.139999) (width 0.4) (layer B.Cu) (net 4))
-  (segment (start 119.38 105.01) (end 119.38 106.68) (width 0.4) (layer B.Cu) (net 4))
-  (segment (start 130.81 96.52) (end 130.81 97.741314) (width 0.4) (layer F.Cu) (net 4))
-  (segment (start 130.81 97.741314) (end 128.221314 100.33) (width 0.4) (layer F.Cu) (net 4))
-  (segment (start 128.221314 100.33) (end 124.46 100.33) (width 0.4) (layer F.Cu) (net 4))
-  (via (at 124.46 100.33) (size 0.6) (drill 0.4) (layers F.Cu B.Cu) (net 4))
-  (segment (start 135.89 96.52) (end 130.81 96.52) (width 0.4) (layer F.Cu) (net 4))
+  (segment (start 119.38 101.981) (end 122.809 105.41) (width 0.5) (layer B.Cu) (net 1))
+  (segment (start 122.809 105.41) (end 127 105.41) (width 0.5) (layer B.Cu) (net 1))
+  (segment (start 129.54 105.41) (end 134.62 105.41) (width 0.5) (layer B.Cu) (net 2))
+  (segment (start 134.62 105.41) (end 135.89 106.68) (width 0.5) (layer B.Cu) (net 2))
+  (segment (start 124.46 96.52) (end 120.142 96.52) (width 0.5) (layer B.Cu) (net 3))
+  (segment (start 120.142 96.52) (end 119.38 97.282) (width 0.5) (layer B.Cu) (net 3))
+  (segment (start 128.27 96.52) (end 124.46 96.52) (width 0.5) (layer F.Cu) (net 3))
+  (via (at 124.46 96.52) (size 1.5) (drill 1) (layers F.Cu B.Cu) (net 3))
+  (segment (start 124.46 107.95) (end 120.65 107.95) (width 0.5) (layer B.Cu) (net 4))
+  (segment (start 120.65 107.95) (end 119.38 106.68) (width 0.5) (layer B.Cu) (net 4))
+  (segment (start 130.81 96.52) (end 130.81 98.479998) (width 0.5) (layer F.Cu) (net 4))
+  (segment (start 130.81 98.479998) (end 124.46 104.829998) (width 0.5) (layer F.Cu) (net 4))
+  (segment (start 124.46 104.829998) (end 124.46 107.95) (width 0.5) (layer F.Cu) (net 4))
+  (via (at 124.46 107.95) (size 1.5) (drill 1) (layers F.Cu B.Cu) (net 4))
+  (segment (start 130.81 96.52) (end 135.89 96.52) (width 0.5) (layer F.Cu) (net 4))
 )
