File: hardware/v1/keys-8.kicad_pcb (KiCad board)
At the start: 2 copper layers, 101 x 32.4 mm, 13 parts, among them P1 CONN_02X02, P2 CONN_01X03, P3 CONN_01X03, P4 CONN_01X03, SW1 SWITCH_INV, SW2 SWITCH_INV, SW3 SWITCH_INV, SW4 SWITCH_INV, SW5 SWITCH_INV, SW6 SWITCH_INV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

Commit message: Re-arrange switch connector pinout to simpler single-row header. Re-route the switch boards accordingly.
Parts:
- P1: value CONN_02X02 -> CONN_01X04; footprint Pin_Headers:Pin_Header_Angled_2x02 -> Pin_Headers:Pin_Header_Angled_1x04
- moved P1 2.54 mm to (229.9, 91.4)
Connections:
- P1 pad 2: /SCK -> VDD
- P1 pad 3: VDD -> /SDA
- P1 pad 4: /SDA -> /SCK
- U1 pad 11: Net-(U1-Pad11) -> (no net)
- U1 pad 14: Net-(U1-Pad14) -> (no net)
- U1 pad 19: Net-(U1-Pad19) -> (no net)
- U1 pad 20: Net-(U1-Pad20) -> (no net)
Routing:
- net /SCK: track 30.5 -> 21.7 mm
- net GND: track 145.9 -> 142.4 mm
- net VDD: track 39.7 -> 42.4 mm
- net /SDA: track 24.9 -> 24.3 mm
