File: hardware/v1/keys-8.sch (KiCad schematic (older format))
At the start: 13 parts, among them P1 CONN_02X02, P2 CONN_01X03, P3 CONN_01X03, P4 CONN_01X03, SW1 SWITCH_INV, SW2 SWITCH_INV, SW3 SWITCH_INV, SW4 SWITCH_INV, SW5 SWITCH_INV, SW6 SWITCH_INV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

Commit message: replace switch footprints on keys-8
Parts:
- SW1, SW2, SW3, SW4, SW5, SW6, SW7, SW8: footprint myparts:SW_SPDT -> myparts:SW_SPDT-custom
Changed lines of the file:
@@
 F 0 "SW1" H 700 1250 50  0000 C CNN
 F 1 "SWITCH_INV" H 750 950 50  0000 C CNN
-F 2 "myparts:SW_SPDT" H 900 1100 50  0001 C CNN
+F 2 "myparts:SW_SPDT-custom" H 900 1100 50  0001 C CNN
 F 3 "" H 900 1100 50  0000 C CNN
 	1    900  1100
@@
 F 0 "SW2" H 1100 1250 50  0000 C CNN
 F 1 "SWITCH_INV" H 1150 950 50  0000 C CNN
-F 2 "myparts:SW_SPDT" H 1300 1100 50  0001 C CNN
+F 2 "myparts:SW_SPDT-custom" H 1300 1100 50  0001 C CNN
 F 3 "" H 1300 1100 50  0000 C CNN
 	1    1300 1100
@@
 F 0 "SW3" H 1500 1250 50  0000 C CNN
 F 1 "SWITCH_INV" H 1550 950 50  0000 C CNN
-F 2 "myparts:SW_SPDT" H 1700 1100 50  0001 C CNN
+F 2 "myparts:SW_SPDT-custom" H 1700 1100 50  0001 C CNN
 F 3 "" H 1700 1100 50  0000 C CNN
 	1    1700 1100
@@
 F 0 "SW4" H 1900 1250 50  0000 C CNN
 F 1 "SWITCH_INV" H 1950 950 50  0000 C CNN
-F 2 "myparts:SW_SPDT" H 2100 1100 50  0001 C CNN
+F 2 "myparts:SW_SPDT-custom" H 2100 1100 50  0001 C CNN
 F 3 "" H 2100 1100 50  0000 C CNN
 	1    2100 1100
@@
 F 0 "SW5" H 2300 1250 50  0000 C CNN
 F 1 "SWITCH_INV" H 2350 950 50  0000 C CNN
-F 2 "myparts:SW_SPDT" H 2500 1100 50  0001 C CNN
+F 2 "myparts:SW_SPDT-custom" H 2500 1100 50  0001 C CNN
 F 3 "" H 2500 1100 50  0000 C CNN
 	1    2500 1100
@@
 F 0 "SW6" H 2700 1250 50  0000 C CNN
 F 1 "SWITCH_INV" H 2750 950 50  0000 C CNN
-F 2 "myparts:SW_SPDT" H 2900 1100 50  0001 C CNN
+F 2 "myparts:SW_SPDT-custom" H 2900 1100 50  0001 C CNN
 F 3 "" H 2900 1100 50  0000 C CNN
 	1    2900 1100
@@
 F 0 "SW7" H 3100 1250 50  0000 C CNN
 F 1 "SWITCH_INV" H 3150 950 50  0000 C CNN
-F 2 "myparts:SW_SPDT" H 3300 1100 50  0001 C CNN
+F 2 "myparts:SW_SPDT-custom" H 3300 1100 50  0001 C CNN
 F 3 "" H 3300 1100 50  0000 C CNN
 	1    3300 1100
@@
 F 0 "SW8" H 3500 1250 50  0000 C CNN
 F 1 "SWITCH_INV" H 3550 950 50  0000 C CNN
-F 2 "myparts:SW_SPDT" H 3700 1100 50  0001 C CNN
+F 2 "myparts:SW_SPDT-custom" H 3700 1100 50  0001 C CNN
 F 3 "" H 3700 1100 50  0000 C CNN
 	1    3700 1100
