File: hardware/v1/switches-16.sch (KiCad schematic (older format))
At the start: 18 parts, among them P1 CONN_02X02, SW1 SWITCH_INV, SW10 SWITCH_INV, SW11 SWITCH_INV, SW12 SWITCH_INV, SW13 SWITCH_INV, SW14 SWITCH_INV, SW15 SWITCH_INV, SW16 SWITCH_INV, SW2 SWITCH_INV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

Commit message: replace switch footprints in switches-16
Parts:
- SW1, SW10, SW11, SW12, SW13, SW14, SW15, SW16, SW2, SW3, SW4, SW5, SW6, SW7, SW8, SW9: footprint myparts:SW_SPDT -> myparts:SW_SPDT-custom
Changed lines of the file:
@@
 F 0 "SW1" H 1300 1650 50  0000 C CNN
 F 1 "SWITCH_INV" H 1350 1350 50  0000 C CNN
-F 2 "myparts:SW_SPDT" H 1500 1500 50  0001 C CNN
+F 2 "myparts:SW_SPDT-custom" H 1500 1500 50  0001 C CNN
 F 3 "" H 1500 1500 50  0000 C CNN
 	1    1500 1500
@@
 F 0 "SW2" H 1800 1650 50  0000 C CNN
 F 1 "SWITCH_INV" H 1850 1350 50  0000 C CNN
-F 2 "myparts:SW_SPDT" H 2000 1500 50  0001 C CNN
+F 2 "myparts:SW_SPDT-custom" H 2000 1500 50  0001 C CNN
 F 3 "" H 2000 1500 50  0000 C CNN
 	1    2000 1500
@@
 F 0 "SW3" H 2250 1650 50  0000 C CNN
 F 1 "SWITCH_INV" H 2300 1350 50  0000 C CNN
-F 2 "myparts:SW_SPDT" H 2450 1500 50  0001 C CNN
+F 2 "myparts:SW_SPDT-custom" H 2450 1500 50  0001 C CNN
 F 3 "" H 2450 1500 50  0000 C CNN
 	1    2450 1500
@@
 F 0 "SW4" H 2700 1650 50  0000 C CNN
 F 1 "SWITCH_INV" H 2750 1350 50  0000 C CNN
-F 2 "myparts:SW_SPDT" H 2900 1500 50  0001 C CNN
+F 2 "myparts:SW_SPDT-custom" H 2900 1500 50  0001 C CNN
 F 3 "" H 2900 1500 50  0000 C CNN
 	1    2900 1500
@@
 F 0 "SW5" H 3200 1650 50  0000 C CNN
 F 1 "SWITCH_INV" H 3250 1350 50  0000 C CNN
-F 2 "myparts:SW_SPDT" H 3400 1500 50  0001 C CNN
+F 2 "myparts:SW_SPDT-custom" H 3400 1500 50  0001 C CNN
 F 3 "" H 3400 1500 50  0000 C CNN
 	1    3400 1500
@@
 F 0 "SW6" H 3700 1650 50  0000 C CNN
 F 1 "SWITCH_INV" H 3750 1350 50  0000 C CNN
-F 2 "myparts:SW_SPDT" H 3900 1500 50  0001 C CNN
+F 2 "myparts:SW_SPDT-custom" H 3900 1500 50  0001 C CNN
 F 3 "" H 3900 1500 50  0000 C CNN
 	1    3900 1500
@@
 F 0 "SW7" H 4150 1650 50  0000 C CNN
 F 1 "SWITCH_INV" H 4200 1350 50  0000 C CNN
-F 2 "myparts:SW_SPDT" H 4350 1500 50  0001 C CNN
+F 2 "myparts:SW_SPDT-custom" H 4350 1500 50  0001 C CNN
 F 3 "" H 4350 1500 50  0000 C CNN
 	1    4350 1500
@@
 F 0 "SW8" H 4600 1650 50  0000 C CNN
 F 1 "SWITCH_INV" H 4650 1350 50  0000 C CNN
-F 2 "myparts:SW_SPDT" H 4800 1500 50  0001 C CNN
+F 2 "myparts:SW_SPDT-custom" H 4800 1500 50  0001 C CNN
 F 3 "" H 4800 1500 50  0000 C CNN
 	1    4800 1500
@@
 F 0 "SW9" H 6750 1650 50  0000 C CNN
 F 1 "SWITCH_INV" H 6800 1350 50  0000 C CNN
-F 2 "myparts:SW_SPDT" H 6950 1500 50  0001 C CNN
+F 2 "myparts:SW_SPDT-custom" H 6950 1500 50  0001 C CNN
 F 3 "" H 6950 1500 50  0000 C CNN
 	1    6950 1500
@@
 F 0 "SW10" H 7250 1650 50  0000 C CNN
 F 1 "SWITCH_INV" H 7300 1350 50  0000 C CNN
-F 2 "myparts:SW_SPDT" H 7450 1500 50  0001 C CNN
+F 2 "myparts:SW_SPDT-custom" H 7450 1500 50  0001 C CNN
 F 3 "" H 7450 1500 50  0000 C CNN
 	1    7450 1500
@@
 F 0 "SW11" H 7700 1650 50  0000 C CNN
 F 1 "SWITCH_INV" H 7750 1350 50  0000 C CNN
-F 2 "myparts:SW_SPDT" H 7900 1500 50  0001 C CNN
+F 2 "myparts:SW_SPDT-custom" H 7900 1500 50  0001 C CNN
 F 3 "" H 7900 1500 50  0000 C CNN
 	1    7900 1500
@@
 F 0 "SW12" H 8150 1650 50  0000 C CNN
 F 1 "SWITCH_INV" H 8200 1350 50  0000 C CNN
-F 2 "myparts:SW_SPDT" H 8350 1500 50  0001 C CNN
+F 2 "myparts:SW_SPDT-custom" H 8350 1500 50  0001 C CNN
 F 3 "" H 8350 1500 50  0000 C CNN
 	1    8350 1500
@@
 F 0 "SW13" H 8650 1650 50  0000 C CNN
 F 1 "SWITCH_INV" H 8700 1350 50  0000 C CNN
-F 2 "myparts:SW_SPDT" H 8850 1500 50  0001 C CNN
+F 2 "myparts:SW_SPDT-custom" H 8850 1500 50  0001 C CNN
 F 3 "" H 8850 1500 50  0000 C CNN
 	1    8850 1500
@@
 F 0 "SW14" H 9150 1650 50  0000 C CNN
 F 1 "SWITCH_INV" H 9200 1350 50  0000 C CNN
-F 2 "myparts:SW_SPDT" H 9350 1500 50  0001 C CNN
+F 2 "myparts:SW_SPDT-custom" H 9350 1500 50  0001 C CNN
 F 3 "" H 9350 1500 50  0000 C CNN
 	1    9350 1500
@@
 F 0 "SW15" H 9600 1650 50  0000 C CNN
 F 1 "SWITCH_INV" H 9650 1350 50  0000 C CNN
-F 2 "myparts:SW_SPDT" H 9800 1500 50  0001 C CNN
+F 2 "myparts:SW_SPDT-custom" H 9800 1500 50  0001 C CNN
 F 3 "" H 9800 1500 50  0000 C CNN
 	1    9800 1500
@@
 F 0 "SW16" H 10050 1650 50  0000 C CNN
 F 1 "SWITCH_INV" H 10100 1350 50  0000 C CNN
-F 2 "myparts:SW_SPDT" H 10250 1500 50  0001 C CNN
+F 2 "myparts:SW_SPDT-custom" H 10250 1500 50  0001 C CNN
 F 3 "" H 10250 1500 50  0000 C CNN
 	1    10250 1500
