File: hardware/v1/lamps-13_3a.sch (KiCad schematic (older format))
At the start: 11 parts, among them P1 CONN_02X05, P2 CONN_01X04, P3 CONN_01X04

Commit message: Replace LED footprints in lamps-13_3a, and delete additional unneded gerber outputs.
Parts:
- D10, D11, D12, D13, D14, D15, D16, D9: footprint LEDs:LED-5MM -> myparts:LED-5MM-custom
Changed lines of the file:
@@
 F 0 "D16" H 6700 6350 50  0000 C CNN
 F 1 "LED" H 6700 6150 50  0000 C CNN
-F 2 "LEDs:LED-5MM" H 6700 6250 50  0001 C CNN
+F 2 "myparts:LED-5MM-custom" H 6700 6250 50  0001 C CNN
 F 3 "" H 6700 6250 50  0000 C CNN
 	1    6700 6250
@@
 F 0 "D15" H 6700 5950 50  0000 C CNN
 F 1 "LED" H 6700 5750 50  0000 C CNN
-F 2 "LEDs:LED-5MM" H 6700 5850 50  0001 C CNN
+F 2 "myparts:LED-5MM-custom" H 6700 5850 50  0001 C CNN
 F 3 "" H 6700 5850 50  0000 C CNN
 	1    6700 5850
@@
 F 0 "D14" H 6700 5550 50  0000 C CNN
 F 1 "LED" H 6700 5350 50  0000 C CNN
-F 2 "LEDs:LED-5MM" H 6700 5450 50  0001 C CNN
+F 2 "myparts:LED-5MM-custom" H 6700 5450 50  0001 C CNN
 F 3 "" H 6700 5450 50  0000 C CNN
 	1    6700 5450
@@
 F 0 "D13" H 4450 4550 50  0000 C CNN
 F 1 "LED" H 4450 4350 50  0000 C CNN
-F 2 "LEDs:LED-5MM" H 4450 4450 50  0001 C CNN
+F 2 "myparts:LED-5MM-custom" H 4450 4450 50  0001 C CNN
 F 3 "" H 4450 4450 50  0000 C CNN
 	1    4450 4450
@@
 F 0 "D12" H 4450 4250 50  0000 C CNN
 F 1 "LED" H 4450 4050 50  0000 C CNN
-F 2 "LEDs:LED-5MM" H 4450 4150 50  0001 C CNN
+F 2 "myparts:LED-5MM-custom" H 4450 4150 50  0001 C CNN
 F 3 "" H 4450 4150 50  0000 C CNN
 	1    4450 4150
@@
 F 0 "D11" H 4450 3850 50  0000 C CNN
 F 1 "LED" H 4450 3650 50  0000 C CNN
-F 2 "LEDs:LED-5MM" H 4450 3750 50  0001 C CNN
+F 2 "myparts:LED-5MM-custom" H 4450 3750 50  0001 C CNN
 F 3 "" H 4450 3750 50  0000 C CNN
 	1    4450 3750
@@
 F 0 "D10" H 4450 3450 50  0000 C CNN
 F 1 "LED" H 4450 3250 50  0000 C CNN
-F 2 "LEDs:LED-5MM" H 4450 3350 50  0001 C CNN
+F 2 "myparts:LED-5MM-custom" H 4450 3350 50  0001 C CNN
 F 3 "" H 4450 3350 50  0000 C CNN
 	1    4450 3350
@@
 F 0 "D9" H 4450 3050 50  0000 C CNN
 F 1 "LED" H 4450 2850 50  0000 C CNN
-F 2 "LEDs:LED-5MM" H 4450 2950 50  0001 C CNN
+F 2 "myparts:LED-5MM-custom" H 4450 2950 50  0001 C CNN
 F 3 "" H 4450 2950 50  0000 C CNN
 	1    4450 2950
