File: hardware/v1/lamps-16.sch (KiCad schematic (older format))
At the start: 1 part, among them P7 CONN_02X05

Commit message: Add keys-8 schematic and initial pcb layout file.
Changed lines of the file:
@@
 $Descr A4 11693 8268
 encoding utf-8
-Sheet 11 25
+Sheet 11 26
 Title "LAMPS-16"
 Date "2016-08-05"
@@
 AR Path="/57A56122/57A3FFF5" Ref="P10"  Part="1"
 AR Path="/57A3FFF5" Ref="P10"  Part="1"
-F 0 "P7" H 1200 1300 50  0000 C CNN
+F 0 "P10" H 1200 1300 50  0000 C CNN
 F 1 "CONN_02X05" H 1200 700 50  0000 C CNN
 F 2 "Pin_Headers:Pin_Header_Angled_2x05" H 1200 -200 50  0001 C CNN

Commit message: Add m3 holes and re-route around them for led boards.
Parts:
- renumbered P7 to P1
Changed lines of the file:
@@
 LIBS:contrib
 LIBS:valves
-LIBS:MAX7221
-LIBS:MCP23S17
-LIBS:MCP23017
-LIBS:Pi2_Connector
-LIBS:v1-cache
+LIBS:lamps-16-cache
 EELAYER 25 0
 EELAYER END
 $Descr A4 11693 8268
 encoding utf-8
-Sheet 11 26
+Sheet 1 3
 Title "LAMPS-16"
 Date "2016-08-05"
@@
 $EndSheet
 $Comp
-L CONN_02X05 P7
+L CONN_02X05 P1
 U 1 1 57A3FFF5
 P 1200 1000
-AR Path="/57A49D32/57A3FFF5" Ref="P7"  Part="1"
-AR Path="/57A54838/57A3FFF5" Ref="P8"  Part="1"
-AR Path="/57A56102/57A3FFF5" Ref="P9"  Part="1"
-AR Path="/57A56122/57A3FFF5" Ref="P10"  Part="1"
-AR Path="/57A3FFF5" Ref="P10"  Part="1"
-F 0 "P10" H 1200 1300 50  0000 C CNN
+F 0 "P1" H 1200 1300 50  0000 C CNN
 F 1 "CONN_02X05" H 1200 700 50  0000 C CNN
 F 2 "Pin_Headers:Pin_Header_Angled_2x05" H 1200 -200 50  0001 C CNN
