File: hardware/v1/ledrow.sch (KiCad schematic (older format))
At the start: 8 parts

Commit message: Replace LED footprints in lamps-13_3a, and delete additional unneded gerber outputs.
Parts:
- D1, D2, D3, D4, D5, D6, D7, D8: footprint LEDs:LED-5MM -> myparts:LED-5MM-custom
Changed lines of the file:
@@
 F 0 "D8" H 1800 4000 50  0000 C CNN
 F 1 "LED" H 1800 3800 50  0000 C CNN
-F 2 "LEDs:LED-5MM" H 1800 3900 50  0001 C CNN
+F 2 "myparts:LED-5MM-custom" H 1800 3900 50  0001 C CNN
 F 3 "" H 1800 3900 50  0000 C CNN
 	1    1800 3900
@@
 F 0 "D7" H 1800 3600 50  0000 C CNN
 F 1 "LED" H 1800 3400 50  0000 C CNN
-F 2 "LEDs:LED-5MM" H 1800 3500 50  0001 C CNN
+F 2 "myparts:LED-5MM-custom" H 1800 3500 50  0001 C CNN
 F 3 "" H 1800 3500 50  0000 C CNN
 	1    1800 3500
@@
 F 0 "D6" H 1800 3200 50  0000 C CNN
 F 1 "LED" H 1800 3000 50  0000 C CNN
-F 2 "LEDs:LED-5MM" H 1800 3100 50  0001 C CNN
+F 2 "myparts:LED-5MM-custom" H 1800 3100 50  0001 C CNN
 F 3 "" H 1800 3100 50  0000 C CNN
 	1    1800 3100
@@
 F 0 "D5" H 1800 2800 50  0000 C CNN
 F 1 "LED" H 1800 2600 50  0000 C CNN
-F 2 "LEDs:LED-5MM" H 1800 2700 50  0001 C CNN
+F 2 "myparts:LED-5MM-custom" H 1800 2700 50  0001 C CNN
 F 3 "" H 1800 2700 50  0000 C CNN
 	1    1800 2700
@@
 F 0 "D4" H 1800 2500 50  0000 C CNN
 F 1 "LED" H 1800 2300 50  0000 C CNN
-F 2 "LEDs:LED-5MM" H 1800 2400 50  0001 C CNN
+F 2 "myparts:LED-5MM-custom" H 1800 2400 50  0001 C CNN
 F 3 "" H 1800 2400 50  0000 C CNN
 	1    1800 2400
@@
 F 0 "D3" H 1800 2100 50  0000 C CNN
 F 1 "LED" H 1800 1900 50  0000 C CNN
-F 2 "LEDs:LED-5MM" H 1800 2000 50  0001 C CNN
+F 2 "myparts:LED-5MM-custom" H 1800 2000 50  0001 C CNN
 F 3 "" H 1800 2000 50  0000 C CNN
 	1    1800 2000
@@
 F 0 "D2" H 1800 1700 50  0000 C CNN
 F 1 "LED" H 1800 1500 50  0000 C CNN
-F 2 "LEDs:LED-5MM" H 1800 1600 50  0001 C CNN
+F 2 "myparts:LED-5MM-custom" H 1800 1600 50  0001 C CNN
 F 3 "" H 1800 1600 50  0000 C CNN
 	1    1800 1600
@@
 F 0 "D1" H 1800 1300 50  0000 C CNN
 F 1 "LED" H 1800 1100 50  0000 C CNN
-F 2 "LEDs:LED-5MM" H 1800 1200 50  0001 C CNN
+F 2 "myparts:LED-5MM-custom" H 1800 1200 50  0001 C CNN
 F 3 "" H 1800 1200 50  0000 C CNN
 	1    1800 1200

Commit message: Add m3 holes and re-route around them for led boards.
Changed lines of the file:
@@
 LIBS:contrib
 LIBS:valves
-LIBS:MAX7221
-LIBS:MCP23S17
-LIBS:MCP23017
-LIBS:Pi2_Connector
-LIBS:v1-cache
+LIBS:lamps-16-cache
 EELAYER 25 0
 EELAYER END
 $Descr A4 11693 8268
 encoding utf-8
-Sheet 12 26
+Sheet 12 3
 Title ""
 Date ""
@@
 U 1 1 57A35AD5
 P 1800 3900
-AR Path="/57A49D32/57A3E922/57A35AD5" Ref="D8"  Part="1"
-AR Path="/57A49D32/57A3F0CE/57A35AD5" Ref="D8"  Part="1"
-AR Path="/57A54838/57A3E922/57A35AD5" Ref="D8"  Part="1"
-AR Path="/57A54838/57A3F0CE/57A35AD5" Ref="D8"  Part="1"
-AR Path="/57A56102/57A3E922/57A35AD5" Ref="D8"  Part="1"
-AR Path="/57A56102/57A3F0CE/57A35AD5" Ref="D8"  Part="1"
-AR Path="/57A56122/57A3E922/57A35AD5" Ref="D8"  Part="1"
-AR Path="/57A56122/57A3F0CE/57A35AD5" Ref="D8"  Part="1"
-AR Path="/57A699EE/57A6A693/57A35AD5" Ref="D8"  Part="1"
-F 0 "D8" H 1800 4000 50  0000 C CNN
+AR Path="/57A3E922/57A35AD5" Ref="D8"  Part="1"
+AR Path="/57A3F0CE/57A35AD5" Ref="D16"  Part="1"
+F 0 "D16" H 1800 4000 50  0000 C CNN
 F 1 "LED" H 1800 3800 50  0000 C CNN
 F 2 "myparts:LED-5MM-custom" H 1800 3900 50  0001 C CNN
@@
 U 1 1 57A35B88
 P 1800 3500
-AR Path="/57A49D32/57A3E922/57A35B88" Ref="D7"  Part="1"
-AR Path="/57A49D32/57A3F0CE/57A35B88" Ref="D7"  Part="1"
-AR Path="/57A54838/57A3E922/57A35B88" Ref="D7"  Part="1"
-AR Path="/57A54838/57A3F0CE/57A35B88" Ref="D7"  Part="1"
-AR Path="/57A56102/57A3E922/57A35B88" Ref="D7"  Part="1"
-AR Path="/57A56102/57A3F0CE/57A35B88" Ref="D7"  Part="1"
-AR Path="/57A56122/57A3E922/57A35B88" Ref="D7"  Part="1"
-AR Path="/57A56122/57A3F0CE/57A35B88" Ref="D7"  Part="1"
-AR Path="/57A699EE/57A6A693/57A35B88" Ref="D7"  Part="1"
-F 0 "D7" H 1800 3600 50  0000 C CNN
+AR Path="/57A3E922/57A35B88" Ref="D7"  Part="1"
+AR Path="/57A3F0CE/57A35B88" Ref="D15"  Part="1"
+F 0 "D15" H 1800 3600 50  0000 C CNN
 F 1 "LED" H 1800 3400 50  0000 C CNN
 F 2 "myparts:LED-5MM-custom" H 1800 3500 50  0001 C CNN
@@
 U 1 1 57A35BB5
 P 1800 3100
-AR Path="/57A49D32/57A3E922/57A35BB5" Ref="D6"  Part="1"
-AR Path="/57A49D32/57A3F0CE/57A35BB5" Ref="D6"  Part="1"
-AR Path="/57A54838/57A3E922/57A35BB5" Ref="D6"  Part="1"
-AR Path="/57A54838/57A3F0CE/57A35BB5" Ref="D6"  Part="1"
-AR Path="/57A56102/57A3E922/57A35BB5" Ref="D6"  Part="1"
-AR Path="/57A56102/57A3F0CE/57A35BB5" Ref="D6"  Part="1"
-AR Path="/57A56122/57A3E922/57A35BB5" Ref="D6"  Part="1"
-AR Path="/57A56122/57A3F0CE/57A35BB5" Ref="D6"  Part="1"
-AR Path="/57A699EE/57A6A693/57A35BB5" Ref="D6"  Part="1"
-F 0 "D6" H 1800 3200 50  0000 C CNN
+AR Path="/57A3E922/57A35BB5" Ref="D6"  Part="1"
+AR Path="/57A3F0CE/57A35BB5" Ref="D14"  Part="1"
+F 0 "D14" H 1800 3200 50  0000 C CNN
 F 1 "LED" H 1800 3000 50  0000 C CNN
 F 2 "myparts:LED-5MM-custom" H 1800 3100 50  0001 C CNN
@@
 U 1 1 57A35BD9
 P 1800 2700
-AR Path="/57A49D32/57A3E922/57A35BD9" Ref="D5"  Part="1"
-AR Path="/57A49D32/57A3F0CE/57A35BD9" Ref="D5"  Part="1"
-AR Path="/57A54838/57A3E922/57A35BD9" Ref="D5"  Part="1"
-AR Path="/57A54838/57A3F0CE/57A35BD9" Ref="D5"  Part="1"
-AR Path="/57A56102/57A3E922/57A35BD9" Ref="D5"  Part="1"
-AR Path="/57A56102/57A3F0CE/57A35BD9" Ref="D5"  Part="1"
-AR Path="/57A56122/57A3E922/57A35BD9" Ref="D5"  Part="1"
-AR Path="/57A56122/57A3F0CE/57A35BD9" Ref="D5"  Part="1"
-AR Path="/57A699EE/57A6A693/57A35BD9" Ref="D5"  Part="1"
-F 0 "D5" H 1800 2800 50  0000 C CNN
+AR Path="/57A3E922/57A35BD9" Ref="D5"  Part="1"
+AR Path="/57A3F0CE/57A35BD9" Ref="D13"  Part="1"
+F 0 "D13" H 1800 2800 50  0000 C CNN
 F 1 "LED" H 1800 2600 50  0000 C CNN
 F 2 "myparts:LED-5MM-custom" H 1800 2700 50  0001 C CNN
@@
 U 1 1 57A35D11
 P 1800 2400
-AR Path="/57A49D32/57A3E922/57A35D11" Ref="D4"  Part="1"
-AR Path="/57A49D32/57A3F0CE/57A35D11" Ref="D4"  Part="1"
-AR Path="/57A54838/57A3E922/57A35D11" Ref="D4"  Part="1"
-AR Path="/57A54838/57A3F0CE/57A35D11" Ref="D4"  Part="1"
-AR Path="/57A56102/57A3E922/57A35D11" Ref="D4"  Part="1"
-AR Path="/57A56102/57A3F0CE/57A35D11" Ref="D4"  Part="1"
-AR Path="/57A56122/57A3E922/57A35D11" Ref="D4"  Part="1"
-AR Path="/57A56122/57A3F0CE/57A35D11" Ref="D4"  Part="1"
-AR Path="/57A699EE/57A6A693/57A35D11" Ref="D4"  Part="1"
-F 0 "D4" H 1800 2500 50  0000 C CNN
+AR Path="/57A3E922/57A35D11" Ref="D4"  Part="1"
+AR Path="/57A3F0CE/57A35D11" Ref="D12"  Part="1"
+F 0 "D12" H 1800 2500 50  0000 C CNN
 F 1 "LED" H 1800 2300 50  0000 C CNN
 F 2 "myparts:LED-5MM-custom" H 1800 2400 50  0001 C CNN
@@
 U 1 1 57A35D17
 P 1800 2000
-AR Path="/57A49D32/57A3E922/57A35D17" Ref="D3"  Part="1"
-AR Path="/57A49D32/57A3F0CE/57A35D17" Ref="D3"  Part="1"
-AR Path="/57A54838/57A3E922/57A35D17" Ref="D3"  Part="1"
-AR Path="/57A54838/57A3F0CE/57A35D17" Ref="D3"  Part="1"
-AR Path="/57A56102/57A3E922/57A35D17" Ref="D3"  Part="1"
-AR Path="/57A56102/57A3F0CE/57A35D17" Ref="D3"  Part="1"
-AR Path="/57A56122/57A3E922/57A35D17" Ref="D3"  Part="1"
-AR Path="/57A56122/57A3F0CE/57A35D17" Ref="D3"  Part="1"
-AR Path="/57A699EE/57A6A693/57A35D17" Ref="D3"  Part="1"
-F 0 "D3" H 1800 2100 50  0000 C CNN
+AR Path="/57A3E922/57A35D17" Ref="D3"  Part="1"
+AR Path="/57A3F0CE/57A35D17" Ref="D11"  Part="1"
+F 0 "D11" H 1800 2100 50  0000 C CNN
 F 1 "LED" H 1800 1900 50  0000 C CNN
 F 2 "myparts:LED-5MM-custom" H 1800 2000 50  0001 C CNN
@@
 U 1 1 57A35D1D
 P 1800 1600
-AR Path="/57A49D32/57A3E922/57A35D1D" Ref="D2"  Part="1"
-AR Path="/57A49D32/57A3F0CE/57A35D1D" Ref="D2"  Part="1"
-AR Path="/57A54838/57A3E922/57A35D1D" Ref="D2"  Part="1"
-AR Path="/57A54838/57A3F0CE/57A35D1D" Ref="D2"  Part="1"
-AR Path="/57A56102/57A3E922/57A35D1D" Ref="D2"  Part="1"
-AR Path="/57A56102/57A3F0CE/57A35D1D" Ref="D2"  Part="1"
-AR Path="/57A56122/57A3E922/57A35D1D" Ref="D2"  Part="1"
-AR Path="/57A56122/57A3F0CE/57A35D1D" Ref="D2"  Part="1"
-AR Path="/57A699EE/57A6A693/57A35D1D" Ref="D2"  Part="1"
-F 0 "D2" H 1800 1700 50  0000 C CNN
+AR Path="/57A3E922/57A35D1D" Ref="D2"  Part="1"
+AR Path="/57A3F0CE/57A35D1D" Ref="D10"  Part="1"
+F 0 "D10" H 1800 1700 50  0000 C CNN
 F 1 "LED" H 1800 1500 50  0000 C CNN
 F 2 "myparts:LED-5MM-custom" H 1800 1600 50  0001 C CNN
@@
 U 1 1 57A35D23
 P 1800 1200
-AR Path="/57A49D32/57A3E922/57A35D23" Ref="D1"  Part="1"
-AR Path="/57A49D32/57A3F0CE/57A35D23" Ref="D1"  Part="1"
-AR Path="/57A54838/57A3E922/57A35D23" Ref="D1"  Part="1"
-AR Path="/57A54838/57A3F0CE/57A35D23" Ref="D1"  Part="1"
-AR Path="/57A56102/57A3E922/57A35D23" Ref="D1"  Part="1"
-AR Path="/57A56102/57A3F0CE/57A35D23" Ref="D1"  Part="1"
-AR Path="/57A56122/57A3E922/57A35D23" Ref="D1"  Part="1"
-AR Path="/57A56122/57A3F0CE/57A35D23" Ref="D1"  Part="1"
-AR Path="/57A699EE/57A6A693/57A35D23" Ref="D1"  Part="1"
-F 0 "D1" H 1800 1300 50  0000 C CNN
+AR Path="/57A3E922/57A35D23" Ref="D1"  Part="1"
+AR Path="/57A3F0CE/57A35D23" Ref="D9"  Part="1"
+F 0 "D9" H 1800 1300 50  0000 C CNN
 F 1 "LED" H 1800 1100 50  0000 C CNN
 F 2 "myparts:LED-5MM-custom" H 1800 1200 50  0001 C CNN
