File: hardware/v1/ledrow.sch (KiCad schematic (older format))
At the start: 8 parts

Commit message: Add pcbs and cutouts for magnetic drum store status lamps (not labelled).
Changed lines of the file:
@@
 LIBS:contrib
 LIBS:valves
-LIBS:MAX7221
-LIBS:MCP23S17
-LIBS:MCP23017
-LIBS:Pi2_Connector
-LIBS:v1-cache
 EELAYER 25 0
 EELAYER END
 $Descr A4 11693 8268
 encoding utf-8
-Sheet 12 31
+Sheet 34 3
 Title ""
 Date ""
@@
 U 1 1 57A35AD5
 P 1800 3900
-AR Path="/57A49D32/57A3E922/57A35AD5" Ref="D8"  Part="1"
-AR Path="/57A49D32/57A3F0CE/57A35AD5" Ref="D16"  Part="1"
-AR Path="/57A54838/57A3E922/57A35AD5" Ref="D24"  Part="1"
-AR Path="/57A54838/57A3F0CE/57A35AD5" Ref="D32"  Part="1"
-AR Path="/57A56102/57A3E922/57A35AD5" Ref="D40"  Part="1"
-AR Path="/57A56102/57A3F0CE/57A35AD5" Ref="D48"  Part="1"
-AR Path="/57A56122/57A3E922/57A35AD5" Ref="D56"  Part="1"
-AR Path="/57A56122/57A3F0CE/57A35AD5" Ref="D64"  Part="1"
-AR Path="/57A699EE/57A6A693/57A35AD5" Ref="D80"  Part="1"
-F 0 "D80" H 1800 4000 50  0000 C CNN
+AR Path="/57AC805C/57A35AD5" Ref="D8"  Part="1"
+AR Path="/57AC8082/57A35AD5" Ref="D16"  Part="1"
+F 0 "D8" H 1800 4000 50  0000 C CNN
 F 1 "LED" H 1800 3800 50  0000 C CNN
 F 2 "myparts:LED-5MM-custom" H 1800 3900 50  0001 C CNN
@@
 U 1 1 57A35B88
 P 1800 3500
-AR Path="/57A49D32/57A3E922/57A35B88" Ref="D7"  Part="1"
-AR Path="/57A49D32/57A3F0CE/57A35B88" Ref="D15"  Part="1"
-AR Path="/57A54838/57A3E922/57A35B88" Ref="D23"  Part="1"
-AR Path="/57A54838/57A3F0CE/57A35B88" Ref="D31"  Part="1"
-AR Path="/57A56102/57A3E922/57A35B88" Ref="D39"  Part="1"
-AR Path="/57A56102/57A3F0CE/57A35B88" Ref="D47"  Part="1"
-AR Path="/57A56122/57A3E922/57A35B88" Ref="D55"  Part="1"
-AR Path="/57A56122/57A3F0CE/57A35B88" Ref="D63"  Part="1"
-AR Path="/57A699EE/57A6A693/57A35B88" Ref="D79"  Part="1"
-F 0 "D79" H 1800 3600 50  0000 C CNN
+AR Path="/57AC805C/57A35B88" Ref="D7"  Part="1"
+AR Path="/57AC8082/57A35B88" Ref="D15"  Part="1"
+F 0 "D7" H 1800 3600 50  0000 C CNN
 F 1 "LED" H 1800 3400 50  0000 C CNN
 F 2 "myparts:LED-5MM-custom" H 1800 3500 50  0001 C CNN
@@
 U 1 1 57A35BB5
 P 1800 3100
-AR Path="/57A49D32/57A3E922/57A35BB5" Ref="D6"  Part="1"
-AR Path="/57A49D32/57A3F0CE/57A35BB5" Ref="D14"  Part="1"
-AR Path="/57A54838/57A3E922/57A35BB5" Ref="D22"  Part="1"
-AR Path="/57A54838/57A3F0CE/57A35BB5" Ref="D30"  Part="1"
-AR Path="/57A56102/57A3E922/57A35BB5" Ref="D38"  Part="1"
-AR Path="/57A56102/57A3F0CE/57A35BB5" Ref="D46"  Part="1"
-AR Path="/57A56122/57A3E922/57A35BB5" Ref="D54"  Part="1"
-AR Path="/57A56122/57A3F0CE/57A35BB5" Ref="D62"  Part="1"
-AR Path="/57A699EE/57A6A693/57A35BB5" Ref="D78"  Part="1"
-F 0 "D78" H 1800 3200 50  0000 C CNN
+AR Path="/57AC805C/57A35BB5" Ref="D6"  Part="1"
+AR Path="/57AC8082/57A35BB5" Ref="D14"  Part="1"
+F 0 "D6" H 1800 3200 50  0000 C CNN
 F 1 "LED" H 1800 3000 50  0000 C CNN
 F 2 "myparts:LED-5MM-custom" H 1800 3100 50  0001 C CNN
@@
 U 1 1 57A35BD9
 P 1800 2700
-AR Path="/57A49D32/57A3E922/57A35BD9" Ref="D5"  Part="1"
-AR Path="/57A49D32/57A3F0CE/57A35BD9" Ref="D13"  Part="1"
-AR Path="/57A54838/57A3E922/57A35BD9" Ref="D21"  Part="1"
-AR Path="/57A54838/57A3F0CE/57A35BD9" Ref="D29"  Part="1"
-AR Path="/57A56102/57A3E922/57A35BD9" Ref="D37"  Part="1"
-AR Path="/57A56102/57A3F0CE/57A35BD9" Ref="D45"  Part="1"
-AR Path="/57A56122/57A3E922/57A35BD9" Ref="D53"  Part="1"
-AR Path="/57A56122/57A3F0CE/57A35BD9" Ref="D61"  Part="1"
-AR Path="/57A699EE/57A6A693/57A35BD9" Ref="D77"  Part="1"
-F 0 "D77" H 1800 2800 50  0000 C CNN
+AR Path="/57AC805C/57A35BD9" Ref="D5"  Part="1"
+AR Path="/57AC8082/57A35BD9" Ref="D13"  Part="1"
+F 0 "D5" H 1800 2800 50  0000 C CNN
 F 1 "LED" H 1800 2600 50  0000 C CNN
 F 2 "myparts:LED-5MM-custom" H 1800 2700 50  0001 C CNN
@@
 U 1 1 57A35D11
 P 1800 2400
-AR Path="/57A49D32/57A3E922/57A35D11" Ref="D4"  Part="1"
-AR Path="/57A49D32/57A3F0CE/57A35D11" Ref="D12"  Part="1"
-AR Path="/57A54838/57A3E922/57A35D11" Ref="D20"  Part="1"
-AR Path="/57A54838/57A3F0CE/57A35D11" Ref="D28"  Part="1"
-AR Path="/57A56102/57A3E922/57A35D11" Ref="D36"  Part="1"
-AR Path="/57A56102/57A3F0CE/57A35D11" Ref="D44"  Part="1"
-AR Path="/57A56122/57A3E922/57A35D11" Ref="D52"  Part="1"
-AR Path="/57A56122/57A3F0CE/57A35D11" Ref="D60"  Part="1"
-AR Path="/57A699EE/57A6A693/57A35D11" Ref="D76"  Part="1"
-F 0 "D76" H 1800 2500 50  0000 C CNN
+AR Path="/57AC805C/57A35D11" Ref="D4"  Part="1"
+AR Path="/57AC8082/57A35D11" Ref="D12"  Part="1"
+F 0 "D4" H 1800 2500 50  0000 C CNN
 F 1 "LED" H 1800 2300 50  0000 C CNN
 F 2 "myparts:LED-5MM-custom" H 1800 2400 50  0001 C CNN
@@
 U 1 1 57A35D17
 P 1800 2000
-AR Path="/57A49D32/57A3E922/57A35D17" Ref="D3"  Part="1"
-AR Path="/57A49D32/57A3F0CE/57A35D17" Ref="D11"  Part="1"
-AR Path="/57A54838/57A3E922/57A35D17" Ref="D19"  Part="1"
-AR Path="/57A54838/57A3F0CE/57A35D17" Ref="D27"  Part="1"
-AR Path="/57A56102/57A3E922/57A35D17" Ref="D35"  Part="1"
-AR Path="/57A56102/57A3F0CE/57A35D17" Ref="D43"  Part="1"
-AR Path="/57A56122/57A3E922/57A35D17" Ref="D51"  Part="1"
-AR Path="/57A56122/57A3F0CE/57A35D17" Ref="D59"  Part="1"
-AR Path="/57A699EE/57A6A693/57A35D17" Ref="D75"  Part="1"
-F 0 "D75" H 1800 2100 50  0000 C CNN
+AR Path="/57AC805C/57A35D17" Ref="D3"  Part="1"
+AR Path="/57AC8082/57A35D17" Ref="D11"  Part="1"
+F 0 "D3" H 1800 2100 50  0000 C CNN
 F 1 "LED" H 1800 1900 50  0000 C CNN
 F 2 "myparts:LED-5MM-custom" H 1800 2000 50  0001 C CNN
@@
 U 1 1 57A35D1D
 P 1800 1600
-AR Path="/57A49D32/57A3E922/57A35D1D" Ref="D2"  Part="1"
-AR Path="/57A49D32/57A3F0CE/57A35D1D" Ref="D10"  Part="1"
-AR Path="/57A54838/57A3E922/57A35D1D" Ref="D18"  Part="1"
-AR Path="/57A54838/57A3F0CE/57A35D1D" Ref="D26"  Part="1"
-AR Path="/57A56102/57A3E922/57A35D1D" Ref="D34"  Part="1"
-AR Path="/57A56102/57A3F0CE/57A35D1D" Ref="D42"  Part="1"
-AR Path="/57A56122/57A3E922/57A35D1D" Ref="D50"  Part="1"
-AR Path="/57A56122/57A3F0CE/57A35D1D" Ref="D58"  Part="1"
-AR Path="/57A699EE/57A6A693/57A35D1D" Ref="D74"  Part="1"
-F 0 "D74" H 1800 1700 50  0000 C CNN
+AR Path="/57AC805C/57A35D1D" Ref="D2"  Part="1"
+AR Path="/57AC8082/57A35D1D" Ref="D10"  Part="1"
+F 0 "D2" H 1800 1700 50  0000 C CNN
 F 1 "LED" H 1800 1500 50  0000 C CNN
 F 2 "myparts:LED-5MM-custom" H 1800 1600 50  0001 C CNN
@@
 U 1 1 57A35D23
 P 1800 1200
-AR Path="/57A49D32/57A3E922/57A35D23" Ref="D1"  Part="1"
-AR Path="/57A49D32/57A3F0CE/57A35D23" Ref="D9"  Part="1"
-AR Path="/57A54838/57A3E922/57A35D23" Ref="D17"  Part="1"
-AR Path="/57A54838/57A3F0CE/57A35D23" Ref="D25"  Part="1"
-AR Path="/57A56102/57A3E922/57A35D23" Ref="D33"  Part="1"
-AR Path="/57A56102/57A3F0CE/57A35D23" Ref="D41"  Part="1"
-AR Path="/57A56122/57A3E922/57A35D23" Ref="D49"  Part="1"
-AR Path="/57A56122/57A3F0CE/57A35D23" Ref="D57"  Part="1"
-AR Path="/57A699EE/57A6A693/57A35D23" Ref="D73"  Part="1"
-F 0 "D73" H 1800 1300 50  0000 C CNN
+AR Path="/57AC805C/57A35D23" Ref="D1"  Part="1"
+AR Path="/57AC8082/57A35D23" Ref="D9"  Part="1"
+F 0 "D1" H 1800 1300 50  0000 C CNN
 F 1 "LED" H 1800 1100 50  0000 C CNN
 F 2 "myparts:LED-5MM-custom" H 1800 1200 50  0001 C CNN
