File: hardware/v1/keys-3-3.sch (KiCad schematic (older format))
At the start: 10 parts, among them P35 CONN_01X04, P36 CONN_01X08, P37 CONN_01X08, SW27 SWITCH_INV, SW28 SWITCH_INV, SW29 SWITCH_INV, U9 MCP23017

Commit message: Integrate first set of switches
Parts:
- renumbered SW29 to CLEAR_ALARM_SW29, CLEAR_ID to CLEAR_ID1, CLEAR_OS to CLEAR_OS1, SW27 to RELEASE_SW27, SPECIAL_WORD to SPECIAL_WORD1, SW28 to STOP_SW28
Changed lines of the file:
@@
 $EndDescr
 $Comp
-L SWITCH_INV SW27
+L SWITCH_INV RELEASE_SW27
 U 1 1 57AB480A
 P 1600 1900
-F 0 "SW27" H 1400 2050 50  0000 C CNN
+F 0 "RELEASE_SW27" H 1400 2050 50  0000 C CNN
 F 1 "SWITCH_INV" H 1450 1750 50  0000 C CNN
 F 2 "myparts:SW_SPDT-custom" H 1600 1900 50  0001 C CNN
@@
 $EndComp
 $Comp
-L SWITCH_INV SW28
+L SWITCH_INV STOP_SW28
 U 1 1 57AB4844
 P 2350 1900
-F 0 "SW28" H 2150 2050 50  0000 C CNN
+F 0 "STOP_SW28" H 2150 2050 50  0000 C CNN
 F 1 "SWITCH_INV" H 2200 1750 50  0000 C CNN
 F 2 "myparts:SW_SPDT-custom" H 2350 1900 50  0001 C CNN
@@
 $EndComp
 $Comp
-L SWITCH_INV SW29
+L SWITCH_INV CLEAR_ALARM_SW29
 U 1 1 57AB4869
 P 3500 1900
-F 0 "SW29" H 3300 2050 50  0000 C CNN
+F 0 "CLEAR_ALARM_SW29" H 3300 2050 50  0000 C CNN
 F 1 "SWITCH_INV" H 3350 1750 50  0000 C CNN
 F 2 "myparts:SW_SPDT-custom" H 3500 1900 50  0001 C CNN
@@
 $EndComp
 $Comp
-L SWITCH_INV CLEAR_OS
+L SWITCH_INV CLEAR_OS1
 U 1 1 57AB4893
 P 8450 3700
-F 0 "CLEAR_OS" H 8250 3850 50  0000 C CNN
+F 0 "CLEAR_OS1" H 8250 3850 50  0000 C CNN
 F 1 "SWITCH_INV" H 8300 3550 50  0000 C CNN
 F 2 "myparts:SW_SPDT-custom" H 8450 3700 50  0001 C CNN
@@
 $EndComp
 $Comp
-L SWITCH_INV CLEAR_ID
+L SWITCH_INV CLEAR_ID1
 U 1 1 57AB48CD
 P 8450 4250
-F 0 "CLEAR_ID" H 8250 4400 50  0000 C CNN
+F 0 "CLEAR_ID1" H 8250 4400 50  0000 C CNN
 F 1 "SWITCH_INV" H 8300 4100 50  0000 C CNN
 F 2 "myparts:SW_SPDT-custom" H 8450 4250 50  0001 C CNN
@@
 $EndComp
 $Comp
-L SWITCH_INV SPECIAL_WORD
+L SWITCH_INV SPECIAL_WORD1
 U 1 1 57AB48F0
 P 8450 5400
-F 0 "SPECIAL_WORD" H 8250 5550 50  0000 C CNN
+F 0 "SPECIAL_WORD1" H 8250 5550 50  0000 C CNN
 F 1 "SWITCH_INV" H 8300 5250 50  0000 C CNN
 F 2 "myparts:SW_SPDT-custom" H 8450 5400 50  0001 C CNN
