File: hardware/v1/keys-6.sch (KiCad schematic (older format))
At the start: 8 parts, among them P38 CONN_01X04, SW33 SWITCH_INV, SW34 SWITCH_INV, SW35 SWITCH_INV, SW36 SWITCH_INV, SW37 SWITCH_INV, SW38 SWITCH_INV, U10 MCP23017

Commit message: Add keys-6 board and add to front panel drawing.
Parts:
- renumbered SW35 to DEST_SW35, SW36 to DISCRIM_SW36, SW33 to NIS_SW33, SW34 to SRC_SW34, SW38 to TCI_SW38, SW37 to TT_SW37
Changed lines of the file:
@@
 LIBS:MCP23017
 LIBS:Pi2_Connector
+LIBS:keys-6-cache
 EELAYER 25 0
 EELAYER END
@@
 $EndDescr
 $Comp
-L SWITCH_INV SW36
+L SWITCH_INV DISCRIM_SW36
 U 1 1 57AB8288
 P 9150 3500
-F 0 "SW36" H 8950 3650 50  0000 C CNN
+F 0 "DISCRIM_SW36" H 8950 3650 50  0000 C CNN
 F 1 "SWITCH_INV" H 9000 3350 50  0000 C CNN
 F 2 "myparts:SW_SPDT-custom" H 9150 3500 50  0001 C CNN
@@
 $EndComp
 $Comp
-L SWITCH_INV SW37
+L SWITCH_INV TT_SW37
 U 1 1 57AB828F
 P 9150 4000
-F 0 "SW37" H 8950 4150 50  0000 C CNN
+F 0 "TT_SW37" H 8950 4150 50  0000 C CNN
 F 1 "SWITCH_INV" H 9000 3850 50  0000 C CNN
 F 2 "myparts:SW_SPDT-custom" H 9150 4000 50  0001 C CNN
@@
 $EndComp
 $Comp
-L SWITCH_INV SW38
+L SWITCH_INV TCI_SW38
 U 1 1 57AB8296
 P 9150 4500
-F 0 "SW38" H 8950 4650 50  0000 C CNN
+F 0 "TCI_SW38" H 8950 4650 50  0000 C CNN
 F 1 "SWITCH_INV" H 9000 4350 50  0000 C CNN
 F 2 "myparts:SW_SPDT-custom" H 9150 4500 50  0001 C CNN
@@
 Connection ~ 9650 4000
 $Comp
-L SWITCH_INV SW33
+L SWITCH_INV NIS_SW33
 U 1 1 57AB8A36
 P 9150 1950
-F 0 "SW33" H 8950 2100 50  0000 C CNN
+F 0 "NIS_SW33" H 8950 2100 50  0000 C CNN
 F 1 "SWITCH_INV" H 9000 1800 50  0000 C CNN
 F 2 "myparts:SW_SPDT-custom" H 9150 1950 50  0001 C CNN
@@
 $EndComp
 $Comp
-L SWITCH_INV SW34
+L SWITCH_INV SRC_SW34
 U 1 1 57AB8A3C
 P 9150 2450
-F 0 "SW34" H 8950 2600 50  0000 C CNN
+F 0 "SRC_SW34" H 8950 2600 50  0000 C CNN
 F 1 "SWITCH_INV" H 9000 2300 50  0000 C CNN
 F 2 "myparts:SW_SPDT-custom" H 9150 2450 50  0001 C CNN
@@
 $EndComp
 $Comp
-L SWITCH_INV SW35
+L SWITCH_INV DEST_SW35
 U 1 1 57AB8A42
 P 9150 2950
-F 0 "SW35" H 8950 3100 50  0000 C CNN
+F 0 "DEST_SW35" H 8950 3100 50  0000 C CNN
 F 1 "SWITCH_INV" H 9000 2800 50  0000 C CNN
 F 2 "myparts:SW_SPDT-custom" H 9150 2950 50  0001 C CNN
