File: hardware/v1/keys-9.sch (KiCad schematic (older format))
At the start: 11 parts, among them P1 CONN_01X04, SW1 SWITCH_INV, SW2 SWITCH_INV, SW3 SWITCH_INV, SW4 SWITCH_INV, SW5 SWITCH_INV, SW6 SWITCH_INV, SW7 SWITCH_INV, SW8 SWITCH_INV, SW9 SWITCH_INV, U1 MCP23017

Commit message: Add Keys-9
Parts:
- renumbered SW1 to SW1_READ1, SW2 to SW2_SINGLE_READ1, SW3 to SW3_PUNCH1, SW4 to SW4_PROGDISP1, SW5 to SW5_TIL1, SW6 to SW6_INIT1, SW7 to SW7_CLEAR1, SW8 to SW8_EXTTREE1, SW9 to SW9_SINGLESHOT1
Connections:
- net PROGDISP_A: now also SW4_PROGDISP1.3; no longer SW4_PROGDISP1.1
- net PROGDISP_B: now also SW4_PROGDISP1.1; no longer SW4_PROGDISP1.3
Changed lines of the file:
@@
 LIBS:MCP23017
 LIBS:Pi2_Connector
+LIBS:keys-9-cache
 EELAYER 25 0
 EELAYER END
@@
 $EndDescr
 $Comp
-L SWITCH_INV SW4
+L SWITCH_INV SW4_PROGDISP1
 U 1 1 57ABB255
 P 8950 3400
-F 0 "SW4" H 8750 3550 50  0000 C CNN
+F 0 "SW4_PROGDISP1" H 8750 3550 50  0000 C CNN
 F 1 "SWITCH_INV" H 8800 3250 50  0000 C CNN
 F 2 "myparts:SW_SPDT-custom" H 8950 3400 50  0001 C CNN
@@
 $EndComp
 $Comp
-L SWITCH_INV SW5
+L SWITCH_INV SW5_TIL1
 U 1 1 57ABB25C
 P 8950 3900
-F 0 "SW5" H 8750 4050 50  0000 C CNN
+F 0 "SW5_TIL1" H 8750 4050 50  0000 C CNN
 F 1 "SWITCH_INV" H 8800 3750 50  0000 C CNN
 F 2 "myparts:SW_SPDT-custom" H 8950 3900 50  0001 C CNN
@@
 $EndComp
 $Comp
-L SWITCH_INV SW6
+L SWITCH_INV SW6_INIT1
 U 1 1 57ABB263
 P 8950 4400
-F 0 "SW6" H 8750 4550 50  0000 C CNN
+F 0 "SW6_INIT1" H 8750 4550 50  0000 C CNN
 F 1 "SWITCH_INV" H 8800 4250 50  0000 C CNN
 F 2 "myparts:SW_SPDT-custom" H 8950 4400 50  0001 C CNN
@@
 Connection ~ 9450 3400
 $Comp
-L GND #PWR4
+L GND #PWR01
 U 1 1 57ABB26D
 P 3100 2850
-F 0 "#PWR4" H 3100 2600 50  0001 C CNN
+F 0 "#PWR01" H 3100 2600 50  0001 C CNN
 F 1 "GND" H 3100 2700 50  0000 C CNN
 F 2 "" H 3100 2850 50  0000 C CNN
@@
 NoConn ~ 4400 3200
 $Comp
-L VDD #PWR3
+L VDD #PWR02
 U 1 1 57ABB279
 P 3100 2650
-F 0 "#PWR3" H 3100 2500 50  0001 C CNN
+F 0 "#PWR02" H 3100 2500 50  0001 C CNN
 F 1 "VDD" H 3100 2800 50  0000 C CNN
 F 2 "" H 3100 2650 50  0000 C CNN
@@
 	3100 2700 3100 2650
 $Comp
-L VDD #PWR2
+L VDD #PWR03
 U 1 1 57ABB283
 P 1250 2150
-F 0 "#PWR2" H 1250 2000 50  0001 C CNN
+F 0 "#PWR03" H 1250 2000 50  0001 C CNN
 F 1 "VDD" H 1250 2300 50  0000 C CNN
 F 2 "" H 1250 2150 50  0000 C CNN
@@
 $EndComp
 $Comp
-L GND #PWR1
+L GND #PWR04
 U 1 1 57ABB289
 P 1250 1750
-F 0 "#PWR1" H 1250 1500 50  0001 C CNN
+F 0 "#PWR04" H 1250 1500 50  0001 C CNN
 F 1 "GND" H 1250 1600 50  0000 C CNN
 F 2 "" H 1250 1750 50  0000 C CNN
@@
 SCK
 $Comp
-L VDD #PWR6
+L VDD #PWR05
 U 1 1 57ABB29D
 P 6300 2850
-F 0 "#PWR6" H 6300 2700 50  0001 C CNN
+F 0 "#PWR05" H 6300 2700 50  0001 C CNN
 F 1 "VDD" H 6300 3000 50  0000 C CNN
 F 2 "" H 6300 2850 50  0000 C CNN
@@
 	6300 2900 5900 2900
 $Comp
-L GND #PWR5
+L GND #PWR06
 U 1 1 57ABB2A5
 P 6100 3350
-F 0 "#PWR5" H 6100 3100 50  0001 C CNN
+F 0 "#PWR06" H 6100 3100 50  0001 C CNN
 F 1 "GND" H 6100 3200 50  0000 C CNN
 F 2 "" H 6100 3350 50  0000 C CNN
@@
 Connection ~ 9450 3900
 $Comp
-L SWITCH_INV SW1
+L SWITCH_INV SW1_READ1
 U 1 1 57ABB2AE
 P 8950 1850
-F 0 "SW1" H 8750 2000 50  0000 C CNN
+F 0 "SW1_READ1" H 8750 2000 50  0000 C CNN
 F 1 "SWITCH_INV" H 8800 1700 50  0000 C CNN
 F 2 "myparts:SW_SPDT-custom" H 8950 1850 50  0001 C CNN
@@
 $EndComp
 $Comp
-L SWITCH_INV SW2
+L SWITCH_INV SW2_SINGLE_READ1
 U 1 1 57ABB2B5
 P 8950 2350
-F 0 "SW2" H 8750 2500 50  0000 C CNN
+F 0 "SW2_SINGLE_READ1" H 8750 2500 50  0000 C CNN
 F 1 "SWITCH_INV" H 8800 2200 50  0000 C CNN
 F 2 "myparts:SW_SPDT-custom" H 8950 2350 50  0001 C CNN
@@
 $EndComp
 $Comp
-L SWITCH_INV SW3
+L SWITCH_INV SW3_PUNCH1
 U 1 1 57ABB2BC
 P 8950 2850
-F 0 "SW3" H 8750 3000 50  0000 C CNN
+F 0 "SW3_PUNCH1" H 8750 3000 50  0000 C CNN
 F 1 "SWITCH_INV" H 8800 2700 50  0000 C CNN
 F 2 "myparts:SW_SPDT-custom" H 8950 2850 50  0001 C CNN
@@
 Text Label 8450 2250 2    60   ~ 0
 SREAD_DOWN
+Text Label 8450 3500 2    60   ~ 0
+PROGDISP_B
 Text Label 8450 3300 2    60   ~ 0
-PROGDISP_B
-Text Label 8450 3500 2    60   ~ 0
 PROGDISP_A
 Text Label 8450 1950 2    60   ~ 0
@@
 INIT_A
 $Comp
-L SWITCH_INV SW7
+L SWITCH_INV SW7_CLEAR1
 U 1 1 57ABB323
 P 8950 4850
-F 0 "SW7" H 8750 5000 50  0000 C CNN
+F 0 "SW7_CLEAR1" H 8750 5000 50  0000 C CNN
 F 1 "SWITCH_INV" H 8800 4700 50  0000 C CNN
 F 2 "myparts:SW_SPDT-custom" H 8950 4850 50  0001 C CNN
@@
 $EndComp
 $Comp
-L SWITCH_INV SW8
+L SWITCH_INV SW8_EXTTREE1
 U 1 1 57ABB353
 P 8950 5300
-F 0 "SW8" H 8750 5450 50  0000 C CNN
+F 0 "SW8_EXTTREE1" H 8750 5450 50  0000 C CNN
 F 1 "SWITCH_INV" H 8800 5150 50  0000 C CNN
 F 2 "myparts:SW_SPDT-custom" H 8950 5300 50  0001 C CNN
@@
 $EndComp
 $Comp
-L SWITCH_INV SW9
+L SWITCH_INV SW9_SINGLESHOT1
 U 1 1 57ABB386
 P 8950 5800
-F 0 "SW9" H 8750 5950 50  0000 C CNN
+F 0 "SW9_SINGLESHOT1" H 8750 5950 50  0000 C CNN
 F 1 "SWITCH_INV" H 8800 5650 50  0000 C CNN
 F 2 "myparts:SW_SPDT-custom" H 8950 5800 50  0001 C CNN
@@
 Connection ~ 9450 5300
 $Comp
-L GND #PWR7
+L GND #PWR07
 U 1 1 57ABB3DD
 P 9450 6100
-F 0 "#PWR7" H 9450 5850 50  0001 C CNN
+F 0 "#PWR07" H 9450 5850 50  0001 C CNN
 F 1 "GND" H 9450 5950 50  0000 C CNN
 F 2 "" H 9450 6100 50  0000 C CNN
